Commit message: new update

File: src/my_robot/urdf/my_robot.urdf (robot description, URDF)
Before this commit: robot ur5_logan, 9 links, 8 joints
Links:
- link base_link: geometry collision mesh filename=file:///home/quocphu/arm6_dof_log/src/my_robot/meshes/base_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; visual mesh filename=file:///home/quocphu/arm6_dof_log/src/my_robot/meshes/base_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
- link ee_link: geometry collision mesh filename=file:///home/quocphu/arm6_dof_log/src/my_robot/meshes/ee_li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; visual mesh filename=file:///home/quocphu/arm6_dof_log/src/my_robot/meshes/ee_li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
- link link1: geometry collision mesh filename=file:///home/quocphu/arm6_dof_log/src/my_robot/meshes/link1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; visual mesh filename=file:///home/quocphu/arm6_dof_log/src/my_robot/meshes/link1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
- link link2: geometry collision mesh filename=file:///home/quocphu/arm6_dof_log/src/my_robot/meshes/link2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; visual mesh filename=file:///home/quocphu/arm6_dof_log/src/my_robot/meshes/link2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
- link link3: geometry collision mesh filename=file:///home/quocphu/arm6_dof_log/src/my_robot/meshes/link3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; visual mesh filename=file:///home/quocphu/arm6_dof_log/src/my_robot/meshes/link3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
- link link4: geometry collision mesh filename=file:///home/quocphu/arm6_dof_log/src/my_robot/meshes/link4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; visual mesh filename=file:///home/quocphu/arm6_dof_log/src/my_robot/meshes/link4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
- link link5: geometry collision mesh filename=file:///home/quocphu/arm6_dof_log/src/my_robot/meshes/link5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; visual mesh filename=file:///home/quocphu/arm6_dof_log/src/my_robot/meshes/link5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
- link link6: geometry collision mesh filename=file:///home/quocphu/arm6_dof_log/src/my_robot/meshes/link6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; visual mesh filename=file:///home/quocphu/arm6_dof_log/src/my_robot/meshes/link6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
